Commit message: Add ugly wheelchair model to rViz

File: jaco_description/robots/standalone_arm.urdf.xacro (robot description, xacro)
@@ -13,8 +13,8 @@
 	xmlns:physics="http://playerstage.sourceforge.net/gazebo/xmlschema/#physics"
 	xmlns:xacro="http://ros.org/wiki/xacro" name="jaco">
-	<xacro:include filename="$(find jaco_description)/urdf/jaco_arm.urdf.xacro" />
+	<xacro:include filename="$(find jaco_description)/urdf/new_model.urdf.xacro" />
 	<link name="root">
 		<visual>
-			<origin xyz="0 0 0" rpy="0 0 0" />
+			<origin xyz="0 0 1" rpy="0 0 0" />
 			<geometry>
 				<box size = "0 0 0" />
@@ -22,5 +22,5 @@
 		</visual>
 		<collision>
-			<origin xyz="0 0 0" rpy="0 0 0" />
+			<origin xyz="0 0 1" rpy="0 0 0" />
 			<geometry>
 				<box size = "0 0 0" />
@@ -28,4 +28,4 @@
 		</collision>
 	</link>
-	<xacro:jaco_arm parent="root" xyz="0 0 0" rpy="0 0 0" />
+	<xacro:jaco_arm parent="root" xyz="0 0 1" rpy="0 0 0" />
 </robot>

Commit message: Create better model

File: jaco_description/robots/standalone_arm.urdf.xacro (robot description, xacro)
@@ -16,5 +16,5 @@
 	<link name="root">
 		<visual>
-			<origin xyz="0 0 1" rpy="0 0 0" />
+			<origin xyz="0 0 0.5" rpy="0 0 0" />
 			<geometry>
 				<box size = "0 0 0" />
@@ -22,5 +22,5 @@
 		</visual>
 		<collision>
-			<origin xyz="0 0 1" rpy="0 0 0" />
+			<origin xyz="0 0 0.5" rpy="0 0 0" />
 			<geometry>
 				<box size = "0 0 0" />
@@ -28,4 +28,4 @@
 		</collision>
 	</link>
-	<xacro:jaco_arm parent="root" xyz="0 0 1" rpy="0 0 0" />
+	<xacro:jaco_arm parent="root" xyz="0 0 0.5" rpy="0 0 0" />
 </robot>

File: jaco_description/urdf/new_model.urdf.xacro (robot description, xacro)
@@ -203,10 +203,10 @@
     <parent link="root"/>
     <child link="base_link"/>
-    <origin xyz="0 0.4 1" rpy="0 0 0" />
+    <origin xyz="0 0.4 0.5" rpy="0 0 0" />
   </joint>
 <link name="base_link">
     <visual>
       <geometry>
-        <box size="0.8 0.7 0.2"/>
+        <box size="0.53 0.52 0.1"/>
       </geometry>
       <origin rpy="0 0 0" xyz="0.0 0 0.1"/>
@@ -218,5 +218,5 @@
     <collision>
       <geometry>
-        <box size="0.8 0.7 0.2"/>
+        <box size="0.53 0.52 0.1"/>
       </geometry>
       <origin rpy="0 0 0" xyz="0.0 0 0.1"/>
@@ -230,5 +230,5 @@
     <visual>
       <geometry>
-        <box size="0.15 0.6 0.8"/>
+        <box size="0.1 0.43 0.52"/>
       </geometry>
       <!--origin rpy="0 0 0" xyz="-0.5 0 0.3"/-->
@@ -239,5 +239,48 @@
     <parent link="base_link"/>
     <child link="back"/>
-    <origin xyz="-0.4 0 0.4"/>
+    <origin xyz="-0.28 0 0.375"/>
+  </joint>
+   <link name="back_head">
+    <visual>
+      <geometry>
+        <box size="0.1 0.23 0.18"/>
+      </geometry>
+      <!--origin rpy="0 0 0" xyz="-0.5 0 0.3"/-->
+      <material name="leather"/>
+    </visual>
+  </link>
+  <joint name="base_link_to_back_head" type="fixed">
+    <parent link="base_link"/>
+    <child link="back_head"/>
+    <origin xyz="-0.28 0 0.7"/>
+  </joint>
+ <!--arm rests-->
+  <link name="arm_rest_right">
+    <visual>
+      <geometry>
+        <box size="0.41 0.07 0.05"/>
+      </geometry>
+      <!--origin rpy="0 0 0" xyz="-0.5 0 0.3"/-->
+      <material name="leather"/>
+    </visual>
+  </link>
+  <joint name="base_link_to_arm_rest_right" type="fixed">
+    <parent link="base_link"/>
+    <child link="arm_rest_right"/>
+    <origin xyz="-0.06 0.24 0.25"/>
+  </joint>
+ <link name="arm_rest_left">
+    <visual>
+      <geometry>
+        <box size="0.41 0.07 0.05"/>
+      </geometry>
+      <!--origin rpy="0 0 0" xyz="-0.5 0 0.3"/-->
+      <material name="leather"/>
+    </visual>
+  </link>
+  <joint name="base_link_to_arm_rest_left" type="fixed">
+    <parent link="base_link"/>
+    <child link="arm_rest_left"/>
+    <origin xyz="-0.06 -0.24 0.25"/>
   </joint>
   <!-- main driving wheels -->
@@ -245,10 +288,9 @@
     <visual>
       <geometry>
-        <cylinder length="0.06" radius="0.12"/>
+        <cylinder length="0.09" radius="0.125"/>
       </geometry>
       <origin rpy="1.57075 0 0" xyz="0.0 0.0 0.0"/>
       <material name="wheel">
         <color rgba="0.0 0.0 0.9 1"/>
-        <!--texture filename="package://jaco_description/urdf/leather.jpg" /-->
       </material>
     </visual>
@@ -263,5 +305,5 @@
     <parent link="base_link"/>
     <child link="left_wheel"/>
-    <origin xyz="0.0 0.35 0.0"/>
+    <origin xyz="0.05 0.3 -0.3"/>
     <axis xyz="0 1 0"/>
   </joint>
@@ -269,5 +311,5 @@
     <visual>
       <geometry>
-        <cylinder length="0.06" radius="0.12"/>
+        <cylinder length="0.09" radius="0.125"/>
       </geometry>
       <origin rpy="1.57075 0 0" xyz="0.0 0.0 0.0"/>
@@ -284,53 +326,48 @@
     <parent link="base_link"/>
     <child link="right_wheel"/>
-    <origin xyz="0.0 -0.35 0.0"/>
+    <origin xyz="0.05 -0.3 -0.3"/>
     <axis xyz="0 1 0"/>
   </joint>
-  <!-- rear castor wheels -->
-  <link name="left_castor">
-    <visual>
-      <geometry>
-        <cylinder length="0.03" radius="0.08"/>
-      </geometry>
-      <origin rpy="1.57075 0 0" xyz="0.0 0.0 0.0"/>
-      <material name="wheel">
-        <color rgba="0.0 0.0 0.9 1"/>
-        <!--texture filename="package://jaco_description/urdf/leather.jpg" /-->
-      </material>
-    </visual>
-    <collision>
-      <geometry>
-        <cylinder length="0.03" radius="0.08"/>
-      </geometry>
-      <origin rpy="1.57075 0 0" xyz="0.0 0.0 0.0"/>
-    </collision>
-  </link>
-  <joint name="base_link_to_left_castor" type="fixed">
-    <parent link="base_link"/>
-    <child link="left_castor"/>
-    <origin xyz="-0.6 0.27 -0.04"/>
-  </joint>
-  <link name="right_castor">
-    <visual>
-      <geometry>
-        <cylinder length="0.03" radius="0.08"/>
-      </geometry>
-      <origin rpy="1.57075 0 0" xyz="0.0 0.0 0.0"/>
-      <material name="wheel">
-        <color rgba="0.0 0.0 0.9 1"/>
-        <!--texture filename="package://jaco_description/urdf/leather.jpg" /-->
-      </material>
-    </visual>
-    <collision>
-      <geometry>
-        <cylinder length="0.03" radius="0.08"/>
-      </geometry>
-      <origin rpy="1.57075 0 0" xyz="0.0 0.0 0.0"/>
-    </collision>
-  </link>
-  <joint name="base_link_to_right_castor" type="fixed">
-    <parent link="base_link"/>
-    <child link="right_castor"/>
-    <origin xyz="-0.6 -0.27 -0.04"/>
+ <link name="motor_cage">
+    <visual>
+      <geometry>
+        <box size="0.48 0.34 0.25"/>
+      </geometry>
+      <!--origin rpy="0 0 0" xyz="-0.5 0 0.3"/-->
+      <material name="leather"/>
+    </visual>
+  </link>
+  <joint name="base_link_to_motor_cage" type="fixed">
+    <parent link="base_link"/>
+    <child link="motor_cage"/>
+    <origin xyz="0 0 -0.2"/>
+  </joint>
+ <link name="under_seat">
+    <visual>
+      <geometry>
+        <box size="0.38 0.32 0.04"/>
+      </geometry>
+      <!--origin rpy="0 0 0" xyz="-0.5 0 0.3"/-->
+      <material name="leather"/>
+    </visual>
+  </link>
+  <joint name="base_link_to_under_seat" type="fixed">
+    <parent link="base_link"/>
+    <child link="under_seat"/>
+    <origin xyz="0 0 0"/>
+  </joint>
+  <link name="foot_plate">
+    <visual>
+      <geometry>
+        <box size="0.44 0.38 0.05"/>
+      </geometry>
+      <!--origin rpy="0 0 0" xyz="-0.5 0 0.3"/-->
+      <material name="leather"/>
+    </visual>
+  </link>
+  <joint name="base_link_to_foot_plate" type="fixed">
+    <parent link="base_link"/>
+    <child link="foot_plate"/>
+    <origin xyz="0.47 0 -0.3"/>
   </joint>
 </robot>

Commit message: Add table model

File: jaco_description/robots/standalone_arm.urdf.xacro (robot description, xacro)
@@ -13,8 +13,8 @@
 	xmlns:physics="http://playerstage.sourceforge.net/gazebo/xmlschema/#physics"
 	xmlns:xacro="http://ros.org/wiki/xacro" name="jaco">
-	<xacro:include filename="$(find jaco_description)/urdf/new_model.urdf.xacro" />
+	<xacro:include filename="$(find jaco_description)/urdf/table_model.urdf.xacro" />
 	<link name="root">
 		<visual>
-			<origin xyz="0 0 0.5" rpy="0 0 0" />
+			<origin xyz="0 0 0.88265" rpy="0 0 0" />
 			<geometry>
 				<box size = "0 0 0" />
@@ -22,5 +22,5 @@
 		</visual>
 		<collision>
-			<origin xyz="0 0 0.5" rpy="0 0 0" />
+			<origin xyz="0 0 0.88265" rpy="0 0 0" />
 			<geometry>
 				<box size = "0 0 0" />
@@ -28,4 +28,4 @@
 		</collision>
 	</link>
-	<xacro:jaco_arm parent="root" xyz="0 0 0.5" rpy="0 0 0" />
+	<xacro:jaco_arm parent="root" xyz="0 0 0.88265" rpy="0 0 0" />
 </robot>
